File: PCB_Design_home/home/home.kicad_sch (KiCad schematic)
At the start: 51 parts, among them J1 USB_C_Receptacle, J2 Conn_01x04_Socket, Q1 2N3904, Q2 2N3904, SW1 SW_Push, SW2 SW_Push, SW3 SW_Push, SW4 SW_Push, U1 AMS1117-3.3, U2 BME680, U3 CP2102N-Axx-xQFN28, U4 ULN2003A, U5 ESP32-C3-WROOM-02

Commit message: Update
Parts:
- removed J1: USB_C_Receptacle, symbol Connector:USB_C_Receptacle
- removed J2: Conn_01x04_Socket, symbol Connector:Conn_01x04_Socket
- added J1: Conn_01x05_Socket, symbol Connector:Conn_01x05_Socket
- added J3: USB_C_Receptacle_USB2.0_16P, Home_Sensor_foot_lib:AMPHENOL_10155435-00011LF, symbol Connector:USB_C_Receptacle_USB2.0_16P
- U3: footprint Package_DFN_QFN:QFN-28-1EP_5x5mm_P0.5mm_EP3.35x3.35mm -> Home_Sensor_foot_lib:QFN50P500X500X80-29N
Connections:
- net +5V: now also J1.1 (Pin_1), J3.A4 (VBUS), J3.A9 (VBUS), J3.B4 (VBUS), J3.B9 (VBUS)
- net GND: now also J3.A1 (GND), J3.A12 (GND), J3.B1 (GND), J3.B12 (GND), J3.S1 (SHIELD)
- net USB_D+: now also J3.A6 (D+), J3.B6 (D+)
- net USB_D-: now also J3.A7 (D-), J3.B7 (D-)
- net at U4.13 (O4): now also J1.5 (Pin_5)
- net at U4.14 (O3): now also J1.4 (Pin_4)
- net at U4.15 (O2): now also J1.3 (Pin_3)
- net at U4.16 (O1): now also J1.2 (Pin_2)
- net at R4.1: now also J3.A5 (CC1)
- net at R5.2: now also J3.B5 (CC2)
- no-connect marks 32 -> 24
Other:
- moved on the sheet: C5, R1, R4, R5
