File: PCB_Design_home/home/home.kicad_sch (KiCad schematic)
At the start: 54 parts, among them J1 USB_C_Receptacle_USB2.0_16P, J2 Conn_01x05_Socket, Q1 2N3904, Q2 2N3904, SW1 SW_Push, SW2 SW_Push, SW3 SW_Push, SW4 SW_Push, U1 ESP32-C3-WROOM-02, U2 CP2102N-Axx-xQFN28, U3 ULN2003A, U4 BME680, U5 AMS1117-3.3

Commit message: Update
Parts:
- removed CR1, CR2, CR3: GG0402052R542P, Home_Sensor_foot_lib:TVS_GG0402_KAV, symbol Hone_Sensor_symbol_lib:GG0402052R542P
- added CR1, CR2, CR3: GG0402052R542P, Home_Sensor_foot_lib:TVS_GG0402_KAV, symbol Home_Sensor_Symbol_lib:GG0402052R542P
- C1, C10, C11, C12, C13, C14, C15, C16, C17, C2, C3, C4, C5, C6, C7, C8, C9: footprint (none) -> Capacitor_SMD:C_0603_1608Metric_Pad1.08x0.95mm_HandSolder
- D1, D2, D3, D4, D5: footprint (none) -> LED_SMD:LED_0603_1608Metric_Pad1.05x0.95mm_HandSolder
- J2: footprint (none) -> Connector_PinSocket_2.54mm:PinSocket_1x05_P2.54mm_Vertical
- R1, R10, R11, R12, R13, R14, R15, R16, R2, R3, R4, R5, R6, R7, R8, R9: footprint (none) -> Resistor_SMD:R_0603_1608Metric_Pad0.98x0.95mm_HandSolder
- SW1, SW2, SW3, SW4: footprint (none) -> Home_Sensor_foot_lib:SW4_1825910-B_TEC
Connections:
- net +5V: now also CR3.1
- net GND: now also CR1.2, CR2.2, CR3.2
- net USB_D+: now also CR1.1
- net USB_D-: now also CR2.1
Other:
- moved on the sheet: C1, R1

Commit message: Update
Parts:
- removed J1: USB_C_Receptacle_USB2.0_16P, Home_Sensor_foot_lib:AMPHENOL_10155435-00011LF, symbol Connector:USB_C_Receptacle_USB2.0_16P
- removed R5: 5.1k, Resistor_SMD:R_0603_1608Metric_Pad0.98x0.95mm_HandSolder, symbol Device:R_Small_US
- removed SW1, SW2, SW3, SW4: SW_Push, Home_Sensor_foot_lib:SW4_1825910-B_TEC, symbol Switch:SW_Push
- added J1: 10155435-00011LF, Home_Sensor_foot_lib:AMPHENOL_10155435-00011LF, symbol Home_Sensor_Symbol_lib:10155435-00011LF
- added R2: 5.1k, Resistor_SMD:R_0603_1608Metric_Pad0.98x0.95mm_HandSolder, symbol Device:R_Small_US
- added SW1, SW2, SW3, SW4: 1825910-6, Home_Sensor_foot_lib:SW4_1825910-B_TEC, symbol Home_Sensor_Symbol_lib:1825910-6
- renumbered R13 to R12, R12 to R13, R2 to R3, R3 to R4, R4 to R5
Connections:
- net +5V: now also CR1.1, J1.A4_B9 (VBUS), J1.B4_A9 (VBUS__1); no longer CR3.1
- net EN: now also C15.2, SW4.3, SW4.4; no longer C14.2
- net GND: now also J1.A1_B12 (GND), J1.B1_A12 (GND__1), J1.SH1 (SHIELD), J1.SH2 (SHIELD__1), J1.SH3 (SHIELD__2), J1.SH4 (SHIELD__3), R2.2, SW1.1, SW1.2, SW2.1, SW2.2, SW3.1, SW3.2, SW4.1, SW4.2
- net IO9: now also C13.2, SW2.3, SW2.4; no longer C15.2
- net Tastknopf1: now also SW1.3, SW1.4
- net Tastknopf2: now also C14.2, SW3.3, SW3.4; no longer C13.2
- net USB_D+: now also CR3.1, J1.A7 (DN1), J1.B6 (DP2); no longer CR1.1
- net USB_D-: now also J1.A6 (DP1), J1.B7 (DN2)
- net at R6.2: now also J1.B5 (CC2)
- new net: J1.A5 (CC1), R2.1
Other:
- moved on the sheet: Q1, Q2, R11, R12

Commit message: Update Display
Parts:
- added C18: 0.1uF, Capacitor_SMD:C_0603_1608Metric_Pad1.08x0.95mm_HandSolder, symbol Device:C_Small
- added J3: Conn_01x04_Socket, Connector_PinSocket_2.54mm:PinSocket_1x04_P2.54mm_Vertical, symbol Connector:Conn_01x04_Socket
Connections:
- net +5V: now also C18.1, J3.3 (Pin_3)
- net GND: now also C18.2, J3.4 (Pin_4)
- net Tastknopf1: now also U1.10 (IO10); no longer U1.13 (IO18)
- net Tastknopf2: no longer U1.14 (IO19)
- new net SCK_display: J3.1 (Pin_1), U1.13 (IO18)
- new net SDA_display: J3.2 (Pin_2), U1.14 (IO19)
- no-connect marks 24 -> 23
Other:
- title: (none) -> Homesensor_Prototyp_v0

Commit message: Temporary placement
Parts:
- removed C14: 0.1uF, Capacitor_SMD:C_0603_1608Metric_Pad1.08x0.95mm_HandSolder, symbol Device:C_Small
- removed SW3: 1825910-6, Home_Sensor_foot_lib:SW4_1825910-B_TEC, symbol Home_Sensor_Symbol_lib:1825910-6
Connections:
- net RXD: now also U1.15 (IO3); no longer U1.12 (IO21/TXD)
- net SCK_display: now also U1.17 (IO1); no longer U1.13 (IO18)
- net SDA_display: now also U1.16 (IO2); no longer U1.14 (IO19)
- net TXD: now also U1.14 (IO19); no longer U1.11 (IO20/RXD)
- net Tastknopf1: now also U1.18 (IO0); no longer U1.10 (IO10)
- net motor1: now also U1.10 (IO10); no longer U1.18 (IO0)
- net motor2: now also U1.11 (IO20/RXD); no longer U1.17 (IO1)
- net motor3: now also U1.12 (IO21/TXD); no longer U1.16 (IO2)
- net motor4: now also U1.13 (IO18); no longer U1.15 (IO3)
Other:
- moved on the sheet: C3, C4, C5, R3

Commit message: Update
Parts:
- removed R1: 1k, Resistor_SMD:R_0603_1608Metric_Pad0.98x0.95mm_HandSolder, symbol Device:R_Small_US
- added C14: 4.7uF, Capacitor_SMD:C_0603_1608Metric_Pad1.08x0.95mm_HandSolder, symbol Device:C_Small
- C1: value 10uF -> 0.1uF
Connections:
- net +3.3V: now also C18.1, J3.3 (Pin_3), C14.1
- net +5V: no longer C18.1, J3.3 (Pin_3)
- net RXD: now also U1.11 (IO20/RXD); no longer U1.15 (IO3)
- net TXD: now also U1.12 (IO21/TXD); no longer U1.14 (IO19)
- net motor2: now also U1.5 (IO6); no longer U1.11 (IO20/RXD)
- net motor3: now also U1.6 (IO7); no longer U1.12 (IO21/TXD)
- net motor4: now also U1.7 (IO8); no longer U1.13 (IO18)
- net at D3.2 (A): now also U1.13 (IO18); no longer U1.7 (IO8)
- net at U2.9 (~{RST}): now also C14.2
- net at D1.2 (A): now also U1.15 (IO3); no longer U1.5 (IO6)
- net at D2.2 (A): now also U1.14 (IO19); no longer U1.6 (IO7)
- net at J2.2 (Pin_2): now also U3.13 (O4); no longer U3.16 (O1)
- net at J2.3 (Pin_3): now also U3.14 (O3); no longer U3.15 (O2)
- net at J2.4 (Pin_4): now also U3.15 (O2); no longer U3.14 (O3)
- net at J2.5 (Pin_5): now also U3.16 (O1); no longer U3.13 (O4)
Other:
- moved on the sheet: C1, D1, D2, D3, R10, R8, R9

Commit message: Testing
Parts:
- removed C14: 4.7uF, Capacitor_SMD:C_0603_1608Metric_Pad1.08x0.95mm_HandSolder, symbol Device:C_Small
- removed C15: 0.1uF, Capacitor_SMD:C_0603_1608Metric_Pad1.08x0.95mm_HandSolder, symbol Device:C_Small
- removed SW4: 1825910-6, Home_Sensor_foot_lib:SW4_1825910-B_TEC, symbol Home_Sensor_Symbol_lib:1825910-6
- added R1: 1k, Resistor_SMD:R_0603_1608Metric_Pad0.98x0.95mm_HandSolder, symbol Device:R_Small_US
- C6: value 0.1uF -> 1uF
- renumbered C16 to C15, C17 to C16, C18 to C17, D3 to D2, D2 to D3, R9 to R10, R10 to R9
Connections:
- net +3.3V: now also R1.2
- net at U2.9 (~{RST}): now also R1.1

Commit message: Testing HW#
Other:
- note added: "io 19 and 18 are swapped in footprint (symbol is wrong)"
Changed lines of the file:
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@@
+		)
+	)
+	(text "io 19 and 18 are swapped in footprint (symbol is wrong)"
+		(exclude_from_sim no)
+		(at 274.32 76.2 0)
+		(effects
+			(font
+				(size 1.27 1.27)
+			)
 		)
 	)
 	(text_box "MCU\n"
 		(exclude_from_sim no)
-		(at 254 16.51 0)
+		(at 243.84 15.24 0)
 		(size 115.57 99.06)
 		(margins 0.9525 0.9525 0.9525 0.9525)
