File: PCB_Design_home/home/_autosave-home.kicad_sch (KiCad schematic)
At the start: 54 parts, among them J1 USB_C_Receptacle_USB2.0_16P, J2 Conn_01x05_Socket, Q1 2N3904, Q2 2N3904, SW1 SW_Push, SW2 SW_Push, SW3 SW_Push, SW4 SW_Push, U1 ESP32-C3-WROOM-02, U2 CP2102N-Axx-xQFN28, U3 ULN2003A, U4 BME680, U5 AMS1117-3.3

Commit message: Update
Parts:
- SW3, SW4: footprint (none) -> Home_Sensor_foot_lib:SW4_1825910-B_TEC
Changed lines of the file:
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@@
 			)
 		)
-		(property "Footprint" ""
+		(property "Footprint" "Home_Sensor_foot_lib:SW4_1825910-B_TEC"
 			(at 36.83 181.61 0)
 			(effects
@@
 			)
 		)
-		(property "Footprint" ""
+		(property "Footprint" "Home_Sensor_foot_lib:SW4_1825910-B_TEC"
 			(at 68.58 181.61 0)
 			(effects
