File: PCB_Design_home/home/home.kicad_pcb (KiCad board)
At the start: 2 copper layers, 54 parts, among them J1 USB_C_Receptacle_USB2.0_16P, J2 Conn_01x05_Socket, Q1 2N3904, Q2 2N3904, SW1 SW_Push, SW2 SW_Push, SW3 SW_Push, SW4 SW_Push, U1 ESP32-C3-WROOM-02, U2 CP2102N-Axx-xQFN28, U3 ULN2003A, U4 BME680, U5 AMS1117-3.3

Commit message: Update
Parts:
- J1: value USB_C_Receptacle_USB2.0_16P -> 10155435-00011LF
- R12: value 4.7k -> 10k
- R13: value 10k -> 4.7k
- R3: value 22.1k -> 5.1k
- R4: value 47.5k -> 22.1k
- R5: value 5.1k -> 47.5k
- SW1, SW2, SW3, SW4: value SW_Push -> 1825910-6
- moved SW1 141.3 mm to (167.4, 67.5)
- moved SW3 134.3 mm to (167.4, 57.2)
- moved SW2 127.0 mm to (141.5, 94.5)
- moved SW4 124.9 mm to (141.5, 105.8)
- moved J2 123.6 mm to (185.8, 74.9)
- moved U3 111.4 mm to (160.9, 76.3)
- moved U2 99.9 mm to (128.8, 67.8)
- moved J1 93.7 mm to (124.3, 106.4), turned to 180 degrees
- moved Q1 82.5 mm to (145.0, 45.0)
- moved Q2 82.5 mm to (145.0, 50.8)
- moved U4 70.8 mm to (104.6, 48.8)
- moved U1 52.8 mm to (127.0, 33.1)
- moved U5 43.4 mm to (112.1, 66.5)
- moved C16 16.3 mm to (45.2, 37.5)
- moved C7 16.3 mm to (40.9, 37.5)
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Connections:
- C13 pad 2: /Tastknopf2 -> /IO9
- C14 pad 2: /EN -> /Tastknopf2
- C15 pad 2: /IO9 -> /EN
- CR1 pad 1: /USB_D+ -> +5V
- CR3 pad 1: +5V -> /USB_D+
- J1 pad A1_B12: (no net) -> GND
- J1 pad A4_B9: (no net) -> +5V
- J1 pad A6: /USB_D+ -> /USB_D-
- J1 pad A7: /USB_D- -> /USB_D+
- J1 pad B1_A12: (no net) -> GND
- J1 pad B4_A9: (no net) -> +5V
- J1 pad SH1: (no net) -> GND
- J1 pad SH2: (no net) -> GND
- J1 pad SH3: (no net) -> GND
- J1 pad SH4: (no net) -> GND
- R12 pad 1: /SCK -> /RTS
- R12 pad 2: +3.3V -> Net-(Q2-B)
- R13 pad 1: /RTS -> /SCK
- R13 pad 2: Net-(Q2-B) -> +3.3V
- R2 pad 1: /EN -> Net-(J1-CC1)
- R2 pad 2: +3.3V -> GND
- R3 pad 1: Net-(U2-VBUS) -> /EN
- R3 pad 2: +5V -> +3.3V
- R4 pad 1: GND -> Net-(U2-VBUS)
- R4 pad 2: Net-(U2-VBUS) -> +5V
- R5 pad 1: Net-(J1-CC1) -> GND
- R5 pad 2: GND -> Net-(U2-VBUS)
- SW1 pad 2: /Tastknopf1 -> GND
- SW1 pad 3: (no net) -> /Tastknopf1
- SW1 pad 4: (no net) -> /Tastknopf1
- SW2 pad 2: /Tastknopf2 -> GND
- SW2 pad 3: (no net) -> /IO9
- SW2 pad 4: (no net) -> /IO9
- SW3 pad 2: /EN -> GND
- SW3 pad 3: (no net) -> /Tastknopf2
- SW3 pad 4: (no net) -> /Tastknopf2
- SW4 pad 2: /IO9 -> GND
- SW4 pad 3: (no net) -> /EN
- SW4 pad 4: (no net) -> /EN

Commit message: Update
Parts:
- moved U3 36.0 mm to (131.2, 56.1)
- moved J2 30.8 mm to (155.0, 74.8)
- moved U4 11.2 mm to (94.6, 53.8)
- moved SW1 7.69 mm to (160.0, 65.3)
- moved SW3 7.69 mm to (160.0, 55.0)
- moved U2 6.87 mm to (124.0, 72.6)
- moved U5 1.49 mm to (112.1, 65.0)
Changed lines of the file:
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@@
 	(footprint "Package_LGA:Bosch_LGA-8_3x3mm_P0.8mm_ClockwisePinNumbering"
 		(layer "F.Cu")
-		(at 104.6 48.8125)
+		(at 94.6 53.8125)
 		(descr "Bosch  LGA, 8 Pin (https://ae-bst.resource.bosch.com/media/_tech/media/datasheets/BST-BME680-DS001-00.pdf#page=44), generated with kicad-footprint-generator ipc_noLead_generator.py")
 		(tags "Bosch LGA NoLead")
@@
 	(footprint "Home_Sensor_foot_lib:SW4_1825910-B_TEC"
 		(layer "F.Cu")
-		(at 167.36 57.2406)
+		(at 160 55)
 		(tags "1825910-6 ")
 		(property "Reference" "SW3"
@@
 	(footprint "Package_TO_SOT_SMD:SOT-223-3_TabPin2"
 		(layer "F.Cu")
-		(at 112.09 66.49)
+		(at 112.09 65)
 		(descr "module CMS SOT223 4 pins")
 		(tags "CMS SOT")
@@
 	(footprint "Home_Sensor_foot_lib:QFN50P500X500X80-29N"
 		(layer "F.Cu")
-		(at 128.83 67.76)
+		(at 124 72.64)
 		(property "Reference" "U2"
 			(at 0.07 -3.94 0)
@@
 	(footprint "Home_Sensor_foot_lib:DIP-16_STM"
 		(layer "F.Cu")
-		(at 160.92 76.3306)
+		(at 131.19 56.11)
 		(tags "ULN2003A ")
 		(property "Reference" "U3"
@@
 	(footprint "Home_Sensor_foot_lib:SW4_1825910-B_TEC"
 		(layer "F.Cu")
-		(at 167.36 67.5106)
+		(at 160 65.27)
 		(tags "1825910-6 ")
 		(property "Reference" "SW1"
@@
 	(footprint "Connector_PinSocket_2.54mm:PinSocket_1x05_P2.54mm_Vertical"
 		(layer "F.Cu")
-		(at 185.78 74.9006)
+		(at 155 74.84)
 		(descr "Through hole straight socket strip, 1x05, 2.54mm pitch, single row (from Kicad 4.0.7), script generated")
 		(tags "Through hole socket strip THT 1x05 2.54mm single row")
@@
 			)
 		)
+	)
+	(zone
+		(net 0)
+		(net_name "")
+		(layer "Edge.Cuts")
+		(hatch edge 0.5)
+		(connect_pads
+			(clearance 0)
+		)
+		(min_thickness 0.25)
+		(filled_areas_thickness no)
+		(keepout
+			(tracks not_allowed)
+			(vias not_allowed)
+			(pads not_allowed)
+			(copperpour allowed)
+			(footprints allowed)
+		)
+		(placement
+			(enabled no)
+			(sheetname "/")
+		)
+		(fill
+			(thermal_gap 0.5)
+			(thermal_bridge_width 0.5)
+		)
+		(polygon
+			(pts
+				(xy 105 15) (xy 150 15) (xy 150 45) (xy 170 45) (xy 170 115) (xy 85 115) (xy 85 45) (xy 105 45)
+			)
+		)

Commit message: Update Display
Parts:
- added C18: 0.1uF, Capacitor_SMD:C_0603_1608Metric_Pad1.08x0.95mm_HandSolder, F.Cu at (77.2, 80.0)
- added J3: Conn_01x04_Socket, Connector_PinSocket_2.54mm:PinSocket_1x04_P2.54mm_Vertical, F.Cu at (125.0, 105.0)
- moved CR3 150.4 mm to (159.4, 117.3)
- moved CR2 150.4 mm to (159.4, 115.0)
- moved CR1 141.4 mm to (139.4, 125.0)
- moved Q1 55.1 mm to (142.5, 100.0)
- moved R8 51.2 mm to (81.6, 77.5)
- moved R11 51.2 mm to (85.9, 62.5)
- moved R13 51.2 mm to (85.9, 67.5)
- moved R14 51.2 mm to (85.9, 70.0)
- moved R16 51.2 mm to (85.9, 75.0)
- moved R2 51.2 mm to (81.6, 62.5)
- moved R4 51.2 mm to (81.6, 67.5)
- moved R5 51.2 mm to (81.6, 70.0)
- moved R7 51.2 mm to (81.6, 75.0)
- moved R12 51.2 mm to (85.9, 65.0)
- moved R15 51.2 mm to (85.9, 72.5)
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Connections:
- U1 pad 10: unconnected-(U1-IO10-Pad10) -> /Tastknopf1
- U1 pad 13: /Tastknopf1 -> /SCK_display
- U1 pad 14: /Tastknopf2 -> /SDA_display

Commit message: Temporary placement
Parts:
- removed C14: 0.1uF, Capacitor_SMD:C_0603_1608Metric_Pad1.08x0.95mm_HandSolder
- removed SW3: 1825910-6, Home_Sensor_foot_lib:SW4_1825910-B_TEC
- moved C8 95.8 mm to (168.3, 86.5)
- moved C15 94.1 mm to (164.4, 107.9)
- moved C7 93.4 mm to (165.8, 84.3)
- moved C12 92.1 mm to (169.0, 57.7), turned to -90 degrees
- moved C18 89.6 mm to (165.9, 92.7)
- moved C13 88.2 mm to (158.9, 100.8)
- moved R6 86.6 mm to (159.9, 109.5), turned to 90 degrees
- moved C2 84.1 mm to (148.3, 99.6), turned to 180 degrees
- moved D4 83.0 mm to (144.4, 101.3), turned to 90 degrees
- moved C6 77.5 mm to (146.4, 97.2)
- moved R2 76.9 mm to (142.4, 109.5), turned to -90 degrees
- moved C1 76.2 mm to (142.1, 91.8), turned to 180 degrees
- moved R1 75.3 mm to (147.9, 95.5)
- moved R7 73.0 mm to (151.6, 95.5)
- moved R5 67.2 mm to (143.0, 97.1)
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Connections:
- U1 pad 10: /Tastknopf1 -> /motor1
- U1 pad 11: /TXD -> /motor2
- U1 pad 12: /RXD -> /motor3
- U1 pad 13: /SCK_display -> /motor4
- U1 pad 14: /SDA_display -> /TXD
- U1 pad 15: /motor4 -> /RXD
- U1 pad 16: /motor3 -> /SDA_display
- U1 pad 17: /motor2 -> /SCK_display
- U1 pad 18: /motor1 -> /Tastknopf1
Routing:
- net /SCK: track 0.00 -> 19.1 mm
- net /SDI: track 0.00 -> 17.9 mm
- net Net-(D1-A): track 0.00 -> 14.9 mm
- net /IO9: track 0.00 -> 14.4 mm
- net +3.3V: track 0.00 -> 11.4 mm
- net Net-(D3-A): track 0.00 -> 11.3 mm
- net Net-(D2-A): track 0.00 -> 11.0 mm
- net GND: track 0.00 -> 10.9 mm, vias 0 -> 8
- net Net-(U2-VBUS): track 0.00 -> 7.31 mm
- net /EN: track 0.00 -> 5.30 mm
- net Net-(D2-K): track 0.00 -> 2.45 mm
- net Net-(D3-K): track 0.00 -> 2.39 mm
- net Net-(D1-K): track 0.00 -> 2.19 mm
- added copper zone on B.Cu, net GND
Other:
- board outline added: 48.2 x 62.3 mm

Commit message: Update
Parts:
- removed R1: 1k, Resistor_SMD:R_0603_1608Metric_Pad0.98x0.95mm_HandSolder
- added C14: 4.7uF, Capacitor_SMD:C_0603_1608Metric_Pad1.08x0.95mm_HandSolder, F.Cu at (229.0, 137.6)
- C1: value 10uF -> 0.1uF
- moved C16 115.4 mm to (196.2, 154.1), turned to -90 degrees
- moved U5 109.2 mm to (193.0, 145.8), turned to 90 degrees
- moved C17 106.2 mm to (187.0, 143.1), turned to -90 degrees
- moved R8 103.7 mm to (228.0, 120.0)
- moved D1 103.3 mm to (228.0, 115.0)
- moved R9 102.0 mm to (226.0, 129.1)
- moved D2 101.6 mm to (226.0, 124.1)
- moved C1 101.0 mm to (233.0, 135.9), turned to 90 degrees
- moved R15 99.1 mm to (184.0, 148.0)
- moved R5 97.9 mm to (230.0, 141.9), turned to 90 degrees
- moved D5 97.8 mm to (184.0, 143.1)
- moved R4 96.8 mm to (227.1, 141.0), turned to 180 degrees
- moved C6 96.6 mm to (232.0, 141.9), turned to -90 degrees
- moved R10 92.2 mm to (224.0, 120.0)
- moved D3 91.8 mm to (224.0, 115.0)
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Connections:
- C18 pad 1: +5V -> +3.3V
- J3 pad 3: +5V -> +3.3V
- U1 pad 11: /motor2 -> /RXD
- U1 pad 12: /motor3 -> /TXD
- U1 pad 13: /motor4 -> Net-(D3-A)
- U1 pad 14: /TXD -> Net-(D2-A)
- U1 pad 15: /RXD -> Net-(D1-A)
- U1 pad 5: Net-(D1-A) -> /motor2
- U1 pad 6: Net-(D2-A) -> /motor3
- U1 pad 7: Net-(D3-A) -> /motor4
- U3 pad 13: Net-(J2-Pin_5) -> Net-(J2-Pin_2)
- U3 pad 14: Net-(J2-Pin_4) -> Net-(J2-Pin_3)
- U3 pad 15: Net-(J2-Pin_3) -> Net-(J2-Pin_4)
- U3 pad 16: Net-(J2-Pin_2) -> Net-(J2-Pin_5)
Routing:
- net +3.3V: track 11.4 -> 247.4 mm
- net +5V: track 0.00 -> 103.1 mm
- net GND: track 10.9 -> 109.2 mm, vias 8 -> 60
- net /EN: track 5.30 -> 66.6 mm, vias 0 -> 5
- net /IO9: track 14.4 -> 63.7 mm, vias 0 -> 3
- net /TXD: track 0.00 -> 31.8 mm, vias 0 -> 2
- net /RXD: track 0.40 -> 31.0 mm, vias 0 -> 2
- net /USB_D-: track 0.00 -> 28.8 mm, vias 0 -> 2
- net /USB_D+: track 0.00 -> 25.7 mm
- net /DTR: track 0.00 -> 23.7 mm
- net /Tastknopf1: track 0.00 -> 23.6 mm
- net /SDA_display: track 0.00 -> 22.1 mm
- net /SCK_display: track 0.00 -> 21.3 mm
- net /RTS: track 0.00 -> 19.1 mm
- net /motor2: track 0.00 -> 19.1 mm
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- added copper zone on F.Cu, net +3.3V
- added copper zone on F.Cu, net +5V
Other:
- board size 48.2 x 62.3 mm -> 60 x 70 mm

Commit message: Update
Other:
- board text added: "HOME SENSOR THE ANH"
Changed lines of the file:
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@@
 			(outputformat 1)
 			(mirror no)
-			(drillshape 1)
+			(drillshape 0)
 			(scaleselection 1)
-			(outputdirectory "")
+			(outputdirectory "../Gerber/")
 		)
 	)
@@
 		(layer "Edge.Cuts")
 	)
+	(gr_text "HOME SENSOR\nTHE ANH"
+		(at 223 155 0)
+		(layer "F.SilkS")
+		(effects
+			(font
+				(size 1 1)
+				(thickness 0.1)
+			)
+			(justify left bottom)
+		)
+	)
 	(segment
 		(start 190.7 150.6)
@@
 				(xy 197.5 103) (xy 197.5 104) (xy 197 104.5) (xy 197 105) (xy 196 106) (xy 192 106) (xy 191.5 105.5)
 				(xy 191.5 99.5) (xy 190.5 98.5) (xy 185 98.5) (xy 184 99.5) (xy 184 124) (xy 186.5 126) (xy 193 126)
-				(xy 193.5 126.5) (xy 193.5 130.5) (xy 193 131) (xy 193.5 133) (xy 195 133.5) (xy 195 133.5) (xy 196 134.5)
-				(xy 196 143.5) (xy 195 144.5) (xy 194 144.5) (xy 194 149) (xy 192.5 151.5) (xy 189 151.5) (xy 188 152.5)
-				(xy 188 156) (xy 188.5 156.5) (xy 230 157)
+				(xy 193.5 126.5) (xy 193.5 130.5) (xy 193 131) (xy 193.5 133) (xy 195 133.5) (xy 196 134.5) (xy 196 143.5)
+				(xy 195 144.5) (xy 194 144.5) (xy 194 149) (xy 192.5 151.5) (xy 189 151.5) (xy 188 152.5) (xy 188 156)
+				(xy 188.5 156.5) (xy 230 157)
 			)
 		)

Commit message: Testing
Parts:
- removed C14: 4.7uF, Capacitor_SMD:C_0603_1608Metric_Pad1.08x0.95mm_HandSolder
- removed C18: 0.1uF, Capacitor_SMD:C_0603_1608Metric_Pad1.08x0.95mm_HandSolder
- removed SW4: 1825910-6, Home_Sensor_foot_lib:SW4_1825910-B_TEC
- added R1: 1k, Resistor_SMD:R_0603_1608Metric_Pad0.98x0.95mm_HandSolder, F.Cu at (229.0, 138.1)
- C15: value 0.1uF -> 22uF
- C17: value 22uF -> 0.1uF
- C6: value 0.1uF -> 1uF
Connections:
- C15 pad 1: GND -> +5V
- C15 pad 2: /EN -> GND
- C16 pad 1: +5V -> +3.3V
- U1 pad 13: Net-(D3-A) -> Net-(D2-A)
- U1 pad 14: Net-(D2-A) -> Net-(D3-A)
Routing:
- net GND: track 109.2 -> 107.6 mm
- net +5V: track 103.1 -> 104.8 mm
